File: elec/layout/default/ldk220m-r.kicad_pcb (KiCad board)
At the start: 2 copper layers, 225.7 x 100.8 mm, 0 parts

Commit message: layout
Parts:
- added C1: Multilayer Ceramic Capacitors MLCC - SMD/SMT 1uF 6.3V 0402 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, lib:C0402, F.Cu at (150.8, 111.6)
- added C2: Multilayer Ceramic Capacitors MLCC - SMD/SMT 1uF 6.3V 0402 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, lib:C0402, F.Cu at (146.4, 111.5)
- added R1: Chip Resistor - Surface Mount 18KOhms ±5% 1/16W 0402 RoHS, lib:R0402, F.Cu at (147.6, 109.2)
- added R2: Chip Resistor - Surface Mount 10KOhms ±5% 1/16W 0402 RoHS, lib:R0402, F.Cu at (149.6, 109.2)
- added U1: , lib:SOT-23-5_L3.0-W1.7-P0.95-LS2.8-BL, F.Cu at (148.6, 111.8)
Routing:
- net gnd: track 0.00 -> 5.62 mm
- net vcc: track 0.00 -> 5.00 mm
- net vcc-1: track 0.00 -> 3.05 mm
- net out: track 0.00 -> 2.56 mm
